File: AryA-Macropad.kicad_pcb (KiCad board)
At the start: 2 copper layers, 37 parts, among them SW1 RotaryEncoder_Switch, SW10 RotaryEncoder_Switch, SW11 SW_SPST, SW12 SW_SPST, SW2 SW_SPST, SW3 SW_SPST, SW4 SW_SPST, SW5 SW_SPST, SW6 SW_SPST, SW7 SW_SPST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

Commit message: Wiring everything up
Parts:
- moved D12 34.1 mm to (180.3, 78.7)
- moved JP11 34.1 mm to (153.0, 73.7)
- moved JP12 34.1 mm to (180.3, 74.9)
- moved JP3 34.1 mm to (153.0, 92.7)
- moved JP7 34.1 mm to (153.0, 111.8)
- moved JP9 34.1 mm to (122.5, 74.9)
- moved SW10 34.1 mm to (168.4, 66.1)
- moved SW12 34.1 mm to (156.2, 68.6)
- moved SW4 34.1 mm to (156.2, 87.6)
- moved SW8 34.1 mm to (156.2, 106.7)
- moved D10 34.1 mm to (133.3, 77.5)
- moved D9 34.1 mm to (122.3, 78.7)
- moved JP1 34.1 mm to (114.9, 92.7)
- moved JP10 34.1 mm to (134.0, 73.7)
- moved JP2 34.1 mm to (134.0, 92.7)
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Connections:
- SW1 pad A: unconnected-(SW1-PadA) -> A1
- SW1 pad B: unconnected-(SW1-PadB) -> B1
- SW1 pad C: unconnected-(SW1-PadC) -> GND
- SW10 pad A: unconnected-(SW10-PadA) -> A2
- SW10 pad B: unconnected-(SW10-PadB) -> B2
- SW10 pad C: unconnected-(SW10-PadC) -> GND
- U1 pad 10: unconnected-(U1-E6-Pad10) -> ROW1
- U1 pad 11: unconnected-(U1-B4-Pad11) -> ROW2
- U1 pad 17: unconnected-(U1-F7-Pad17) -> Net-(U1-F7)
- U1 pad 18: unconnected-(U1-F6-Pad18) -> Net-(U1-F6)
- U1 pad 19: unconnected-(U1-F5-Pad19) -> Net-(U1-F5)
- U1 pad 20: unconnected-(U1-F4-Pad20) -> Net-(U1-F4)
- U1 pad 23: unconnected-(U1-GND-Pad23) -> GND
- U1 pad 5: unconnected-(U1-SDA-Pad5) -> COL0
- U1 pad 6: unconnected-(U1-SCL-Pad6) -> COL1
- U1 pad 7: unconnected-(U1-D4-Pad7) -> COL2
- U1 pad 8: unconnected-(U1-C6-Pad8) -> COL3
- U1 pad 9: unconnected-(U1-D7-Pad9) -> ROW0
Routing:
- net COL3: track 0.00 -> 195.6 mm
- net COL2: track 0.00 -> 180.0 mm
- net ROW0: track 0.00 -> 163.3 mm
- net COL1: track 0.00 -> 159.8 mm
- net ROW1: track 0.00 -> 136.7 mm
- net COL0: track 0.00 -> 134.9 mm
- net ROW2: track 0.00 -> 127.0 mm
- net GND: track 0.00 -> 86.5 mm
- net Net-(D8-A): track 0.00 -> 19.9 mm
- net Net-(D5-A): track 0.00 -> 18.6 mm
- net Net-(D10-A): track 0.00 -> 18.5 mm
- net Net-(D11-A): track 0.00 -> 18.2 mm
- net Net-(D7-A): track 0.00 -> 17.1 mm
- net Net-(D6-A): track 0.00 -> 17.1 mm
- net Net-(D4-A): track 0.00 -> 17.1 mm
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
Commit message: finishing up schematic
Connections:
- U1 pad 10: ROW1 -> COL3
- U1 pad 11: ROW2 -> unconnected-(U1-B4-Pad11)
- U1 pad 14: unconnected-(U1-B2-Pad14) -> ROW2
- U1 pad 15: unconnected-(U1-B3-Pad15) -> ROW1
- U1 pad 16: unconnected-(U1-B1-Pad16) -> ROW0
- U1 pad 21: unconnected-(U1-VCC-Pad21) -> +5V
- U1 pad 5: COL0 -> Net-(J1-Pin_1)
- U1 pad 6: COL1 -> Net-(J1-Pin_2)
- U1 pad 7: COL2 -> COL0
- U1 pad 8: COL3 -> COL1
- U1 pad 9: ROW0 -> COL2
Routing:
- net ROW0: track 163.3 -> 102.4 mm
- net ROW1: track 136.7 -> 102.7 mm
- net ROW2: track 127.0 -> 119.7 mm
- net COL3: track 195.6 -> 190.5 mm
- net COL2: track 180.0 -> 174.9 mm
- net COL1: track 159.8 -> 154.7 mm
- net GND: track 86.5 -> 91.2 mm
- net COL0: track 134.9 -> 130.3 mm

Commit message: 1.0 complete
Parts:
- added H1: MountingHole, MountingHole:MountingHole_2.5mm, F.Cu at (80.2, 64.3)
- added H2: MountingHole, MountingHole:MountingHole_2.5mm, F.Cu at (190.5, 64.3)
- added H3: MountingHole, MountingHole:MountingHole_2.5mm, F.Cu at (80.2, 114.3)
- added H4: MountingHole, MountingHole:MountingHole_2.5mm, F.Cu at (190.5, 114.3)
- added J1: i2c display, Connector_PinHeader_2.54mm:PinHeader_1x04_P2.54mm_Vertical, F.Cu at (99.0, 115.1)
- added R1: 10K, Resistor_SMD:R_1206_3216Metric_Pad1.30x1.75mm_HandSolder, B.Cu at (106.4, 73.0)
- added R2: 10K, Resistor_SMD:R_1206_3216Metric_Pad1.30x1.75mm_HandSolder, B.Cu at (106.4, 67.5)
- added R3: 10K, Resistor_SMD:R_1206_3216Metric_Pad1.30x1.75mm_HandSolder, B.Cu at (165.1, 69.8)
- added R4: 10K, Resistor_SMD:R_1206_3216Metric_Pad1.30x1.75mm_HandSolder, B.Cu at (165.1, 64.3)
- added R5: 10K, Resistor_SMD:R_1206_3216Metric_Pad1.30x1.75mm_HandSolder, B.Cu at (92.1, 71.4)
- added R6: 10K, Resistor_SMD:R_1206_3216Metric_Pad1.30x1.75mm_HandSolder, B.Cu at (98.4, 71.4)
Connections:
- U1 pad 17: Net-(U1-F7) -> B2
- U1 pad 18: Net-(U1-F6) -> A2
- U1 pad 19: Net-(U1-F5) -> B1
- U1 pad 20: Net-(U1-F4) -> A1
Routing:
- net +5V: track 0.00 -> 148.7 mm, vias 0 -> 2
- net B2: track 0.00 -> 82.3 mm
- net A2: track 0.00 -> 75.2 mm
- net Net-(J1-Pin_3): track 0.00 -> 55.6 mm
- net GND: track 91.2 -> 141.7 mm
- net Net-(J1-Pin_4): track 0.00 -> 49.0 mm
- net A1: track 0.00 -> 14.5 mm
- net COL0: track 130.3 -> 144.5 mm
- net COL2: track 174.9 -> 188.9 mm
- net COL3: track 190.5 -> 204.1 mm
- net COL1: track 154.7 -> 168.3 mm
- net B1: track 0.00 -> 8.67 mm
- net Net-(D8-A): track 19.9 -> 12.4 mm
- net Net-(D11-A): track 18.2 -> 12.4 mm
- net Net-(D5-A): track 18.6 -> 12.8 mm
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Other:
- board outline added: 123 x 62.7 mm

Commit message: updated code
Routing:
- net COL3: track 204.1 -> 196.3 mm
Changed lines of the file:
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@@
       (plot_on_all_layers_selection 0x0000000_00000000)
       (disableapertmacros false)
-      (usegerberextensions false)
-      (usegerberattributes true)
-      (usegerberadvancedattributes true)
-      (creategerberjobfile true)
+      (usegerberextensions true)
+      (usegerberattributes false)
+      (usegerberadvancedattributes false)
+      (creategerberjobfile false)
       (dashed_line_dash_ratio 12.000000)
       (dashed_line_gap_ratio 3.000000)
@@
       (psa4output false)
       (plotreference true)
-      (plotvalue true)
+      (plotvalue false)
       (plotinvisibletext false)
       (sketchpadsonfab false)
-      (subtractmaskfromsilk false)
+      (subtractmaskfromsilk true)
       (outputformat 1)
       (mirror false)
-      (drillshape 1)
+      (drillshape 0)
       (scaleselection 1)
-      (outputdirectory "")
+      (outputdirectory "Version 1.0/")
     )
   )
@@
     (fp_line (start 1.6 0.8) (end 1.6 -0.8)
       (stroke (width 0.1) (type solid)) (layer "B.Fab"))
-    (pad "1" smd roundrect (at -1.55 0 270) (size 1.3 1.75) (layers "B.Cu" "B.Paste" "B.Mask") (roundrect_rratio 0.192308)
+    (pad "1" smd roundrect (at -1.55 0 270) (size 1.3 1.75) (layers "B.Cu" "B.Paste" "B.Mask") (roundrect_rratio 0.1923076923)
       (net 23 "B2") (pintype "passive"))
-    (pad "2" smd roundrect (at 1.55 0 270) (size 1.3 1.75) (layers "B.Cu" "B.Paste" "B.Mask") (roundrect_rratio 0.192308)
+    (pad "2" smd roundrect (at 1.55 0 270) (size 1.3 1.75) (layers "B.Cu" "B.Paste" "B.Mask") (roundrect_rratio 0.1923076923)
       (net 34 "+5V") (pintype "passive"))
     (model "${KICAD6_3DMODEL_DIR}/Resistor_SMD.3dshapes/R_1206_3216Metric.wrl"
@@
     (fp_line (start 1.6 0.8) (end 1.6 -0.8)
       (stroke (width 0.1) (type solid)) (layer "B.Fab"))
-    (pad "1" smd roundrect (at -1.55 0 90) (size 1.3 1.75) (layers "B.Cu" "B.Paste" "B.Mask") (roundrect_rratio 0.192308)
+    (pad "1" smd roundrect (at -1.55 0 90) (size 1.3 1.75) (layers "B.Cu" "B.Paste" "B.Mask") (roundrect_rratio 0.1923076923)
       (net 18 "A1") (pintype "passive"))
-    (pad "2" smd roundrect (at 1.55 0 90) (size 1.3 1.75) (layers "B.Cu" "B.Paste" "B.Mask") (roundrect_rratio 0.192308)
+    (pad "2" smd roundrect (at 1.55 0 90) (size 1.3 1.75) (layers "B.Cu" "B.Paste" "B.Mask") (roundrect_rratio 0.1923076923)
       (net 34 "+5V") (pintype "passive"))
     (model "${KICAD6_3DMODEL_DIR}/Resistor_SMD.3dshapes/R_1206_3216Metric.wrl"
@@
     (fp_line (start 1.6 0.8) (end 1.6 -0.8)
       (stroke (width 0.1) (type solid)) (layer "B.Fab"))
-    (pad "1" smd roundrect (at -1.55 0 90) (size 1.3 1.75) (layers "B.Cu" "B.Paste" "B.Mask") (roundrect_rratio 0.192308)
+    (pad "1" smd roundrect (at -1.55 0 90) (size 1.3 1.75) (layers "B.Cu" "B.Paste" "B.Mask") (roundrect_rratio 0.1923076923)
       (net 32 "Net-(J1-Pin_4)") (pintype "passive"))
-    (pad "2" smd roundrect (at 1.55 0 90) (size 1.3 1.75) (layers "B.Cu" "B.Paste" "B.Mask") (roundrect_rratio 0.192308)
+    (pad "2" smd roundrect (at 1.55 0 90) (size 1.3 1.75) (layers "B.Cu" "B.Paste" "B.Mask") (roundrect_rratio 0.1923076923)
       (net 34 "+5V") (pintype "passive"))
     (model "${KICAD6_3DMODEL_DIR}/Resistor_SMD.3dshapes/R_1206_3216Metric.wrl"
@@
     (fp_line (start 1.6 0.8) (end 1.6 -0.8)
       (stroke (width 0.1) (type solid)) (layer "B.Fab"))
-    (pad "1" smd roundrect (at -1.55 0 90) (size 1.3 1.75) (layers "B.Cu" "B.Paste" "B.Mask") (roundrect_rratio 0.192308)
+    (pad "1" smd roundrect (at -1.55 0 90) (size 1.3 1.75) (layers "B.Cu" "B.Paste" "B.Mask") (roundrect_rratio 0.1923076923)
       (net 31 "Net-(J1-Pin_3)") (pintype "passive"))
-    (pad "2" smd roundrect (at 1.55 0 90) (size 1.3 1.75) (layers "B.Cu" "B.Paste" "B.Mask") (roundrect_rratio 0.192308)
+    (pad "2" smd roundrect (at 1.55 0 90) (size 1.3 1.75) (layers "B.Cu" "B.Paste" "B.Mask") (roundrect_rratio 0.1923076923)
       (net 34 "+5V") (pintype "passive"))
     (model "${KICAD6_3DMODEL_DIR}/Resistor_SMD.3dshapes/R_1206_3216Metric.wrl"
@@
     (fp_line (start 1.6 0.8) (end 1.6 -0.8)
       (stroke (width 0.1) (type solid)) (layer "B.Fab"))
-    (pad "1" smd roundrect (at -1.55 0 270) (size 1.3 1.75) (layers "B.Cu" "B.Paste" "B.Mask") (roundrect_rratio 0.192308)
+    (pad "1" smd roundrect (at -1.55 0 270) (size 1.3 1.75) (layers "B.Cu" "B.Paste" "B.Mask") (roundrect_rratio 0.1923076923)
       (net 24 "A2") (pintype "passive"))
-    (pad "2" smd roundrect (at 1.55 0 270) (size 1.3 1.75) (layers "B.Cu" "B.Paste" "B.Mask") (roundrect_rratio 0.192308)
+    (pad "2" smd roundrect (at 1.55 0 270) (size 1.3 1.75) (layers "B.Cu" "B.Paste" "B.Mask") (roundrect_rratio 0.1923076923)
       (net 34 "+5V") (pintype "passive"))
     (model "${KICAD6_3DMODEL_DIR}/Resistor_SMD.3dshapes/R_1206_3216Metric.wrl"
@@
     (fp_line (start 1.6 0.8) (end 1.6 -0.8)
       (stroke (width 0.1) (type solid)) (layer "B.Fab"))
-    (pad "1" smd roundrect (at -1.55 0 90) (size 1.3 1.75) (layers "B.Cu" "B.Paste" "B.Mask") (roundrect_rratio 0.192308)
+    (pad "1" smd roundrect (at -1.55 0 90) (size 1.3 1.75) (layers "B.Cu" "B.Paste" "B.Mask") (roundrect_rratio 0.1923076923)
       (net 17 "B1") (pintype "passive"))
-    (pad "2" smd roundrect (at 1.55 0 90) (size 1.3 1.75) (layers "B.Cu" "B.Paste" "B.Mask") (roundrect_rratio 0.192308)
+    (pad "2" smd roundrect (at 1.55 0 90) (size 1.3 1.75) (layers "B.Cu" "B.Paste" "B.Mask") (roundrect_rratio 0.1923076923)
       (net 34 "+5V") (pintype "passive"))
     (model "${KICAD6_3DMODEL_DIR}/Resistor_SMD.3dshapes/R_1206_3216Metric.wrl"
@@
   (segment (start 164.30625 104.61625) (end 164.30625 104.775) (width 0.25) (layer "F.Cu") (net 21))
   (segment (start 181.61 82.55) (end 182.88 83.82) (width 0.25) (layer "F.Cu") (net 22))
-  (segment (start 172.24375 78.58125) (end 176.2125 82.55) (width 0.25) (layer "F.Cu") (net 22))
-  (segment (start 172.24375 71.4375) (end 172.24375 78.58125) (width 0.25) (layer "F.Cu") (net 22))
-  (segment (start 177.56125 66.12) (end 172.24375 71.4375) (width 0.25) (layer "F.Cu") (net 22))
+  (segment (start 184.94375 68.18375) (end 182.88 66.12) (width 0.25) (layer "F.Cu") (net 22))
   (segment (start 182.88 96.52) (end 177.8 101.6) (width 0.25) (layer "F.Cu") (net 22))
   (segment (start 182.88 96.52) (end 182.88 114.3) (width 0.25) (layer "F.Cu") (net 22))
   (segment (start 84.93125 116.68125) (end 84.93125 87.78875) (width 0.25) (layer "F.Cu") (net 22))
-  (segment (start 176.2125 82.55) (end 177.8 82.55) (width 0.25) (layer "F.Cu") (net 22))
+  (segment (start 182.88 83.82) (end 184.94375 81.75625) (width 0.25) (layer "F.Cu") (net 22))
+  (segment (start 184.94375 81.75625) (end 184.94375 68.18375) (width 0.25) (layer "F.Cu") (net 22))
   (segment (start 87.3125 119.0625) (end 84.93125 116.68125) (width 0.25) (layer "F.Cu") (net 22))
   (segment (start 178.1175 119.0625) (end 87.3125 119.0625) (width 0.25) (layer "F.Cu") (net 22))
   (segment (start 84.93125 87.78875) (end 87.63 85.09) (width 0.25) (layer "F.Cu") (net 22))
   (segment (start 182.88 114.3) (end 178.1175 119.0625) (width 0.25) (layer "F.Cu") (net 22))
-  (segment (start 182.88 66.12) (end 177.56125 66.12) (width 0.25) (layer "F.Cu") (net 22))
   (segment (start 182.88 83.82) (end 182.88 96.52) (width 0.25) (layer "F.Cu") (net 22))
   (segment (start 177.8 82.55) (end 181.61 82.55) (width 0.25) (layer "F.Cu") (net 22))
