File: AryA-Macropad.kicad_sch (KiCad schematic)
At the start: 37 parts, among them SW1 RotaryEncoder_Switch, SW10 RotaryEncoder_Switch, SW11 SW_SPST, SW12 SW_SPST, SW2 SW_SPST, SW3 SW_SPST, SW4 SW_SPST, SW5 SW_SPST, SW6 SW_SPST, SW7 SW_SPST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

Commit message: Wiring everything up
Parts:
- added R1, R2, R3, R4: 10K, symbol Device:R
Connections:
- net COL0: now also U1.5 (SDA)
- net COL1: now also U1.6 (SCL)
- net COL2: now also U1.7 (D4)
- net COL3: now also U1.8 (C6)
- net ROW0: now also U1.9 (D7)
- net ROW1: now also U1.10 (E6)
- net ROW2: now also U1.11 (B4)
- net at U1.17 (F7): now also R3.1
- net at U1.18 (F6): now also R4.1
- net at U1.19 (F5): now also R1.1
- net at U1.20 (F4): now also R2.1
- net GND: now reaches U1.23 (GND)
- net GND: now also SW1.C, SW10.C
- net A1: now reaches SW1.A
- net A1: now also R2.2
- net B1: now reaches SW1.B
- net B1: now also R1.2
- net A2: now reaches SW10.A
- net A2: now also R4.2
- net B2: now reaches SW10.B
- net B2: now also R3.2
Other:
- title: (none) -> Macro Pad
- moved on the sheet: U1

Commit message: finishing up schematic
Parts:
- added H1, H2, H3, H4: MountingHole, symbol Mechanical:MountingHole
- added J1: i2c display, symbol Connector:Conn_01x04_Socket
- added R5, R6: 10K, symbol Device:R
Connections:
- net COL0: now also U1.7 (D4); no longer U1.5 (SDA)
- net COL1: now also U1.8 (C6); no longer U1.6 (SCL)
- net COL2: now also U1.9 (D7); no longer U1.7 (D4)
- net COL3: now also U1.10 (E6); no longer U1.8 (C6)
- net GND: now also J1.4 (Pin_4)
- net ROW0: now also U1.16 (B1); no longer U1.9 (D7)
- net ROW1: now also U1.15 (B3); no longer U1.10 (E6)
- net ROW2: now also U1.14 (B2); no longer U1.11 (B4)
- net +5V: now reaches U1.21 (VCC)
- net +5V: now also J1.3 (Pin_3), R5.2, R6.2
- new net: J1.1 (Pin_1), R5.1, U1.5 (SDA)
- new net: J1.2 (Pin_2), R6.1, U1.6 (SCL)
Other:
- moved on the sheet: D1, D10, D11, D12, D2, D3, D4, D5, D6, D7, D8, D9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

Commit message: 1.0 complete
Parts:
- H1, H2, H3, H4: footprint (none) -> MountingHole:MountingHole_2.5mm
- J1: footprint (none) -> Connector_PinHeader_2.54mm:PinHeader_1x04_P2.54mm_Vertical
- R1, R2, R3, R4, R5, R6: footprint (none) -> Resistor_SMD:R_1206_3216Metric_Pad1.30x1.75mm_HandSolder
Connections:
- net +5V: now also J1.2 (Pin_2), R1.2, R2.2, R3.2, R4.2; no longer J1.3 (Pin_3)
- net A1: now also R2.1, U1.20 (F4); no longer R2.2
- net A2: now also R4.1, U1.18 (F6); no longer R4.2
- net B1: now also R1.1, U1.19 (F5); no longer R1.2
- net B2: now also R3.1, U1.17 (F7); no longer R3.2
- net GND: now also J1.1 (Pin_1); no longer J1.4 (Pin_4)
- net at R5.1, U1.5 (SDA): now also J1.4 (Pin_4); no longer J1.1 (Pin_1)
- net at R6.1, U1.6 (SCL): now also J1.3 (Pin_3); no longer J1.2 (Pin_2)
Other:
- moved on the sheet: J1, R1, R2, R3, R4

Commit message: small changes
Parts:
- removed R5, R6: 10K, Resistor_SMD:R_1206_3216Metric_Pad1.30x1.75mm_HandSolder, symbol Device:R
Changed lines of the file:
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@@
   (junction (at 250.19 128.27) (diameter 0) (color 0 0 0 0)
   )
-  (junction (at 34.29 111.76) (diameter 0) (color 0 0 0 0)
-  )
   (junction (at 220.98 109.22) (diameter 0) (color 0 0 0 0)
   )
@@
   (junction (at 220.98 78.74) (diameter 0) (color 0 0 0 0)
   )
-  (junction (at 31.75 118.11) (diameter 0) (color 0 0 0 0)
-  )
   (junction (at 191.77 128.27) (diameter 0) (color 0 0 0 0)
   )
@@
   (junction (at 162.56 138.43) (diameter 0) (color 0 0 0 0)
   )
-  (wire (pts (xy 44.45 111.76) (xy 46.99 111.76))
-    (stroke (width 0) (type default))
-  )
   (wire (pts (xy 147.32 62.23) (xy 147.32 63.5))
     (stroke (width 0) (type default))
@@
     (stroke (width 0) (type default))
   )
-  (wire (pts (xy 34.29 111.76) (xy 36.83 111.76))
-    (stroke (width 0) (type default))
-  )
   (wire (pts (xy 250.19 90.17) (xy 250.19 96.52))
     (stroke (width 0) (type default))
@@
     (stroke (width 0) (type default))
   )
-  (wire (pts (xy 31.75 118.11) (xy 31.75 132.08))
+  (wire (pts (xy 31.75 85.09) (xy 31.75 132.08))
     (stroke (width 0) (type default))
   )
@@
     (stroke (width 0) (type default))
   )
-  (wire (pts (xy 31.75 118.11) (xy 46.99 118.11))
-    (stroke (width 0) (type default))
-  )
   (wire (pts (xy 153.67 128.27) (xy 162.56 128.27))
     (stroke (width 0) (type default))
@@
     (stroke (width 0) (type default))
   )
-  (wire (pts (xy 46.99 111.76) (xy 46.99 107.95))
-    (stroke (width 0) (type default))
-  )
   (wire (pts (xy 220.98 78.74) (xy 250.19 78.74))
     (stroke (width 0) (type default))
@@
     (stroke (width 0) (type default))
   )
-  (wire (pts (xy 34.29 111.76) (xy 34.29 132.08))
-    (stroke (width 0) (type default))
-  )
   (wire (pts (xy 48.26 95.25) (xy 49.53 95.25))
     (stroke (width 0) (type default))
@@
     (stroke (width 0) (type default))
   )
-  (wire (pts (xy 54.61 118.11) (xy 57.15 118.11))
-    (stroke (width 0) (type default))
-  )
   (wire (pts (xy 191.77 109.22) (xy 220.98 109.22))
     (stroke (width 0) (type default))
@@
     (stroke (width 0) (type default))
   )
-  (wire (pts (xy 34.29 82.55) (xy 34.29 111.76))
+  (wire (pts (xy 34.29 82.55) (xy 34.29 132.08))
     (stroke (width 0) (type default))
   )
@@
     (stroke (width 0) (type default))
   )
-  (wire (pts (xy 57.15 118.11) (xy 57.15 115.57))
-    (stroke (width 0) (type default))
-  )
   (wire (pts (xy 191.77 74.93) (xy 191.77 73.66))
     (stroke (width 0) (type default))
@@
   )
   (wire (pts (xy 182.88 138.43) (xy 191.77 138.43))
-    (stroke (width 0) (type default))
-  )
-  (wire (pts (xy 31.75 85.09) (xy 31.75 118.11))
     (stroke (width 0) (type default))
   )
@@
     (property "Intersheetrefs" "${INTERSHEET_REFS}" (at 201.93 37.8967 90)
       (effects (font (size 1.27 1.27)) (justify left) hide)
-    )
-  )
-  (symbol (lib_id "Device:R") (at 40.64 111.76 90) (unit 1)
-    (in_bom yes) (on_board yes) (dnp no) (fields_autoplaced)
-    (property "Reference" "R5" (at 40.64 105.41 90)
-      (effects (font (size 1.27 1.27)))
-    )
-    (property "Value" "10K" (at 40.64 107.95 90)
-      (effects (font (size 1.27 1.27)))
-    )
-    (property "Footprint" "Resistor_SMD:R_1206_3216Metric_Pad1.30x1.75mm_HandSolder" (at 40.64 113.538 90)
-      (effects (font (size 1.27 1.27)) hide)
-    )
-    (property "Datasheet" "~" (at 40.64 111.76 0)
-      (effects (font (size 1.27 1.27)) hide)
-    )
-    (pin "2")
-    (pin "1")
-    (instances
-      (project "AryA-Macropad"
-        (path "/49354fbe-b562-4be7-a56b-d8466f40604d"
-          (reference "R5") (unit 1)
-        )
-      )
     )
   )
@@
     )
   )
-  (symbol (lib_id "power:+5V") (at 57.15 115.57 0) (unit 1)
-    (in_bom yes) (on_board yes) (dnp no) (fields_autoplaced)
-    (property "Reference" "#PWR08" (at 57.15 119.38 0)
-      (effects (font (size 1.27 1.27)) hide)
-    )
-    (property "Value" "+5V" (at 57.15 110.49 0)
-      (effects (font (size 1.27 1.27)))
-    )
-    (property "Footprint" "" (at 57.15 115.57 0)
-      (effects (font (size 1.27 1.27)) hide)
-    )
-    (property "Datasheet" "" (at 57.15 115.57 0)
-      (effects (font (size 1.27 1.27)) hide)
-    )
-    (pin "1")
-    (instances
-      (project "AryA-Macropad"
-        (path "/49354fbe-b562-4be7-a56b-d8466f40604d"
-          (reference "#PWR08") (unit 1)
-        )
-      )
-    )
-  )
   (symbol (lib_id "Device:R") (at 114.3 85.09 90) (unit 1)
     (in_bom yes) (on_board yes) (dnp no) (fields_autoplaced)
@@
         (path "/49354fbe-b562-4be7-a56b-d8466f40604d"
           (reference "JP7") (unit 1)
-        )
-      )
-    )
-  )
-  (symbol (lib_id "power:+5V") (at 46.99 107.95 0) (unit 1)
-    (in_bom yes) (on_board yes) (dnp no) (fields_autoplaced)
-    (property "Reference" "#PWR07" (at 46.99 111.76 0)
-      (effects (font (size 1.27 1.27)) hide)
-    )
-    (property "Value" "+5V" (at 46.99 102.87 0)
-      (effects (font (size 1.27 1.27)))
-    )
-    (property "Footprint" "" (at 46.99 107.95 0)
-      (effects (font (size 1.27 1.27)) hide)
-    )
-    (property "Datasheet" "" (at 46.99 107.95 0)
-      (effects (font (size 1.27 1.27)) hide)
-    )
-    (pin "1")
-    (instances
-      (project "AryA-Macropad"
-        (path "/49354fbe-b562-4be7-a56b-d8466f40604d"
-          (reference "#PWR07") (unit 1)
         )
       )
@@
         )
       )
-    )
-  )
-  (symbol (lib_id "Device:R") (at 50.8 118.11 90) (unit 1)
-    (in_bom yes) (on_board yes) (dnp no) (fields_autoplaced)
-    (property "Reference" "R6" (at 50.8 111.76 90)
-      (effects (font (size 1.27 1.27)))
-    )
-    (property "Value" "10K" (at 50.8 114.3 90)
-      (effects (font (size 1.27 1.27)))
-    )
-    (property "Footprint" "Resistor_SMD:R_1206_3216Metric_Pad1.30x1.75mm_HandSolder" (at 50.8 119.888 90)
-      (effects (font (size 1.27 1.27)) hide)
-    )
-    (property "Datasheet" "~" (at 50.8 118.11 0)
-      (effects (font (size 1.27 1.27)) hide)
-    )
-    (pin "2")
-    (pin "1")
-    (instances
-      (project "AryA-Macropad"
-        (path "/49354fbe-b562-4be7-a56b-d8466f40604d"
-          (reference "R6") (unit 1)
-        )
-      )
